File: arduino-theremin/v1/arduino-theremin-v1.kicad_pcb (KiCad board)
At the start: 2 copper layers, 71.1 x 53.3 mm, 15 parts, among them SW2 ON-OFF-ON SWITCH, U1 Arduino_Uno_R3_Shield

Commit message: Not actually sure about this commit...
Parts:
- removed RESET: SW_PUSH, Buttons_Switches_ThroughHole:SW_TH_Tactile_Omron_B3F-10xx
- added SW1: SW_PUSH_B3F_1XXX, Buttons_Switches_ThroughHole:SW_TH_Tactile_Omron_B3F-10xx, F.Cu at (125.7, 102.9)
Routing:
- net /RESET: track 14.2 -> 16.3 mm
- net +5V: track 69.2 -> 70.5 mm
Other:
- board text added: "Arduino Theremin Shield Demo Board v1.1 OSH Park 2016"
- board text removed: "Arduino Theremin Shield Demo Board v1.0 OSH Park 2016"
Changed lines of the file:
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@@
   )
   (setup
-    (last_trace_width 0.508)
+    (last_trace_width 0.254)
     (user_trace_width 0.1524)
     (user_trace_width 0.254)
@@
     )
   )
+  (module Wicker_Buttons_Switches:ESwitch_Series100_SPDT (layer F.Cu)
+    (at 91.44 102.87 90)
+    (descr "Three-position through-hole board mount switch.")
+    (tags "ON-OFF-ON switch")
+    (fp_text reference SW2 (at 0 -5.1 90) (layer F.SilkS) hide
+      (effects (font (size 1 1) (thickness 0.15)))
+    )
+    (fp_text value "ON-OFF-ON SWITCH" (at 0 -3.1 90) (layer F.Fab)
+      (effects (font (size 1 1) (thickness 0.15)))
+    )
+    (fp_line (start -1.55 0) (end -1.55 -1.55) (layer F.SilkS) (width 0.15))
+    (fp_line (start -1.55 -1.55) (end 1.55 -1.55) (layer F.SilkS) (width 0.15))
+    (fp_line (start 1.55 -1.55) (end 1.55 0) (layer F.SilkS) (width 0.15))
+    (fp_line (start -1.75 -1.75) (end -1.75 11.43) (layer F.CrtYd) (width 0.05))
+    (fp_line (start 1.75 -1.75) (end 1.75 11.43) (layer F.CrtYd) (width 0.05))
+    (fp_line (start -1.75 -1.75) (end 1.75 -1.75) (layer F.CrtYd) (width 0.05))
+    (fp_line (start -1.75 11.43) (end 1.75 11.43) (layer F.CrtYd) (width 0.05))
+    (fp_line (start 1.27 1.27) (end 1.27 10.922) (layer F.SilkS) (width 0.15))
+    (fp_line (start 1.27 10.922) (end -1.27 10.922) (layer F.SilkS) (width 0.15))
+    (fp_line (start -1.27 10.922) (end -1.27 1.27) (layer F.SilkS) (width 0.15))
+    (pad 1 thru_hole rect (at 0 0 90) (size 2.032 1.7272) (drill 1.016) (layers *.Cu *.Mask F.SilkS)
+      (net 9 /D9_BTN_RECORD))
+    (pad 2 thru_hole oval (at 0 4.699 90) (size 2.032 1.7272) (drill 1.016) (layers *.Cu *.Mask F.SilkS)
+      (net 1 +5V))
+    (pad 3 thru_hole oval (at 0 9.398 90) (size 2.032 1.7272) (drill 1.016) (layers *.Cu *.Mask F.SilkS)
+      (net 8 /D8_BTN_PLAYBACK))
+  )
   (module Buttons_Switches_ThroughHole:SW_TH_Tactile_Omron_B3F-10xx (layer F.Cu)
-    (at 124.968 103.124)
+    (at 125.73 102.87)
     (descr SW_TH_Tactile_Omron_B3F-10xx)
     (tags "Omron B3F-10xx")
-    (fp_text reference RESET (at 8.89 1.778 90) (layer F.SilkS)
-      (effects (font (size 1.27 1.27) (thickness 0.254)))
-    )
-    (fp_text value SW_PUSH (at 2.95 -2.05) (layer F.Fab)
+    (fp_text reference SW1 (at 3 6) (layer F.SilkS)
+      (effects (font (size 1 1) (thickness 0.15)))
+    )
+    (fp_text value SW_PUSH_B3F_1XXX (at 2.95 -2.05) (layer F.Fab)
       (effects (font (size 1 1) (thickness 0.15)))
     )
@@
     (fp_circle (center 3 2) (end 4 3) (layer F.SilkS) (width 0))
     (pad 4 thru_hole circle (at 6 4) (size 1.7 1.7) (drill 1) (layers *.Cu *.Mask))
-    (pad 3 thru_hole circle (at 0 4) (size 1.7 1.7) (drill 1) (layers *.Cu *.Mask))
-    (pad 2 thru_hole circle (at 6 0) (size 1.7 1.7) (drill 1) (layers *.Cu *.Mask)
-      (net 2 GND))
+    (pad 3 thru_hole circle (at 0 4) (size 1.7 1.7) (drill 1) (layers *.Cu *.Mask)
+      (net 2 GND))
+    (pad 2 thru_hole circle (at 6 0) (size 1.7 1.7) (drill 1) (layers *.Cu *.Mask))
     (pad 1 thru_hole circle (at 0 0) (size 1.7 1.7) (drill 1) (layers *.Cu *.Mask)
       (net 7 /RESET))
   )
-  (module Wicker_Buttons_Switches:ESwitch_Series100_SPDT (layer F.Cu)
-    (at 91.44 102.87 90)
-    (descr "Three-position through-hole board mount switch.")
-    (tags "ON-OFF-ON switch")
-    (fp_text reference SW2 (at 0 -5.1 90) (layer F.SilkS) hide
-      (effects (font (size 1 1) (thickness 0.15)))
-    )
-    (fp_text value "ON-OFF-ON SWITCH" (at 0 -3.1 90) (layer F.Fab)
-      (effects (font (size 1 1) (thickness 0.15)))
-    )
-    (fp_line (start -1.55 0) (end -1.55 -1.55) (layer F.SilkS) (width 0.15))
-    (fp_line (start -1.55 -1.55) (end 1.55 -1.55) (layer F.SilkS) (width 0.15))
-    (fp_line (start 1.55 -1.55) (end 1.55 0) (layer F.SilkS) (width 0.15))
-    (fp_line (start -1.75 -1.75) (end -1.75 11.43) (layer F.CrtYd) (width 0.05))
-    (fp_line (start 1.75 -1.75) (end 1.75 11.43) (layer F.CrtYd) (width 0.05))
-    (fp_line (start -1.75 -1.75) (end 1.75 -1.75) (layer F.CrtYd) (width 0.05))
-    (fp_line (start -1.75 11.43) (end 1.75 11.43) (layer F.CrtYd) (width 0.05))
-    (fp_line (start 1.27 1.27) (end 1.27 10.922) (layer F.SilkS) (width 0.15))
-    (fp_line (start 1.27 10.922) (end -1.27 10.922) (layer F.SilkS) (width 0.15))
-    (fp_line (start -1.27 10.922) (end -1.27 1.27) (layer F.SilkS) (width 0.15))
-    (pad 1 thru_hole rect (at 0 0 90) (size 2.032 1.7272) (drill 1.016) (layers *.Cu *.Mask F.SilkS)
-      (net 9 /D9_BTN_RECORD))
-    (pad 2 thru_hole oval (at 0 4.699 90) (size 2.032 1.7272) (drill 1.016) (layers *.Cu *.Mask F.SilkS)
-      (net 1 +5V))
-    (pad 3 thru_hole oval (at 0 9.398 90) (size 2.032 1.7272) (drill 1.016) (layers *.Cu *.Mask F.SilkS)
-      (net 8 /D8_BTN_PLAYBACK))
-  )
-  (gr_text "Arduino Theremin Shield \nDemo Board v1.0\n\nOSH Park 2016" (at 140.208 91.186 90) (layer B.SilkS)
+  (gr_text "Arduino Theremin Shield \nDemo Board v1.1\n\nOSH Park 2016" (at 140.208 91.186 90) (layer B.SilkS)
     (effects (font (size 1.5 1.5) (thickness 0.3)) (justify mirror))
   )
@@
   (gr_line (start 120.523 82.55) (end 120.523 93.98) (angle 90) (layer Dwgs.User) (width 0.15))
   (gr_line (start 104.648 82.55) (end 120.523 82.55) (angle 90) (layer Dwgs.User) (width 0.15))
+  (segment (start 113.284 90.678) (end 123.698 101.346) (width 0.508) (layer B.Cu) (net 1))
+  (segment (start 123.698 101.346) (end 128.016 101.346) (width 0.508) (layer B.Cu) (net 1))
+  (segment (start 128.016 101.346) (end 128.27 101.6) (width 0.508) (layer B.Cu) (net 1))
+  (segment (start 128.27 101.6) (end 128.27 109.22) (width 0.508) (layer B.Cu) (net 1))
+  (segment (start 128.27 109.22) (end 125.73 111.76) (width 0.508) (layer B.Cu) (net 1))
+  (segment (start 125.73 111.76) (end 125.73 115.57) (width 0.508) (layer B.Cu) (net 1))
   (segment (start 125.7935 92.7735) (end 125.5395 92.7735) (width 0.508) (layer F.Cu) (net 1))
   (segment (start 113.284 90.678) (end 121.666 90.678) (width 0.762) (layer F.Cu) (net 1))
@@
   (segment (start 121.666 90.678) (end 123.7615 92.7735) (width 0.762) (layer F.Cu) (net 1))
   (via (at 113.284 90.678) (size 0.6858) (drill 0.3302) (layers F.Cu B.Cu) (net 1))
-  (segment (start 123.698 101.346) (end 113.284 90.678) (width 0.508) (layer B.Cu) (net 1))
-  (segment (start 128.016 104.14) (end 126.492 101.346) (width 0.508) (layer B.Cu) (net 1))
-  (segment (start 126.492 101.346) (end 123.698 101.346) (width 0.508) (layer B.Cu) (net 1))
-  (segment (start 128.016 104.902) (end 128.016 104.14) (width 0.508) (layer B.Cu) (net 1))
-  (segment (start 128.016 109.474) (end 128.016 104.902) (width 0.508) (layer B.Cu) (net 1))
-  (segment (start 126.326001 111.163999) (end 128.016 109.474) (width 0.508) (layer B.Cu) (net 1))
-  (segment (start 125.73 111.76) (end 126.326001 111.163999) (width 0.508) (layer B.Cu) (net 1))
-  (segment (start 125.73 115.57) (end 125.73 111.76) (width 0.508) (layer B.Cu) (net 1))
   (segment (start 112.268 90.678) (end 113.284 90.678) (width 0.508) (layer F.Cu) (net 1))
   (segment (start 125.5395 92.7735) (end 125.476 92.71) (width 0.508) (layer F.Cu) (net 1))
@@
   (segment (start 102.616 109.728) (end 141.478 109.728) (width 0.508) (layer F.Cu) (net 6))
   (via (at 141.478 109.728) (size 0.6858) (drill 0.3302) (layers F.Cu B.Cu) (net 6))
+  (segment (start 123.19 102.87) (end 120.65 105.41) (width 0.508) (layer B.Cu) (net 7))
+  (segment (start 120.65 105.41) (end 120.65 107.442) (width 0.508) (layer B.Cu) (net 7))
+  (segment (start 125.73 102.87) (end 123.19 102.87) (width 0.508) (layer B.Cu) (net 7))
   (segment (start 120.65 115.57) (end 120.65 107.442) (width 0.508) (layer B.Cu) (net 7))
-  (segment (start 120.65 107.442) (end 124.968 103.124) (width 0.508) (layer B.Cu) (net 7))
   (segment (start 97.536 80.518) (end 101.2825 80.518) (width 0.508) (layer B.Cu) (net 8))
   (segment (start 98.552 105.156) (end 98.298 105.41) (width 0.508) (layer B.Cu) (net 8))
