File: arduino-theremin/v1/arduino-theremin-v1.sch (KiCad schematic (older format))
At the start: 15 parts, among them P1 LV-EZ1 RANGEFINDER, SW1 SW_PUSH, SW2 ON-OFF-ON SWITCH, U1 Arduino_Uno_R3_Shield

Commit message: Not actually sure about this commit...
Parts:
- removed SW1: SW_PUSH, Buttons_Switches_ThroughHole:SW_TH_Tactile_Omron_B3F-10xx, symbol SW_PUSH
- added SW?: SW_PUSH_B3F_1XXX, symbol SW_PUSH_B3F_1XXX
Connections:
- net GND: now also SW?.3
- net RESET: now also SW?.1
- no-connect marks 21 -> 23
Changed lines of the file:
@@
 D5_KEY3
 $Comp
-L +5V #PWR01
+L +5V #PWR3
 U 1 1 56B18B8A
 P 2800 1575
-F 0 "#PWR01" H 2800 1425 50  0001 C CNN
+F 0 "#PWR3" H 2800 1425 50  0001 C CNN
 F 1 "+5V" H 2800 1715 50  0000 C CNN
 F 2 "" H 2800 1575 50  0000 C CNN
@@
 $EndComp
 $Comp
-L +5V #PWR02
+L +5V #PWR14
 U 1 1 56BD38C1
 P 9225 1575
-F 0 "#PWR02" H 9225 1425 50  0001 C CNN
+F 0 "#PWR14" H 9225 1425 50  0001 C CNN
 F 1 "+5V" H 9225 1715 50  0000 C CNN
 F 2 "" H 9225 1575 50  0000 C CNN
@@
 $EndComp
 $Comp
-L GND #PWR03
+L GND #PWR8
 U 1 1 56BD4329
 P 7675 2275
-F 0 "#PWR03" H 7675 2025 50  0001 C CNN
+F 0 "#PWR8" H 7675 2025 50  0001 C CNN
 F 1 "GND" H 7675 2125 50  0000 C CNN
 F 2 "" H 7675 2275 50  0000 C CNN
@@
 $EndComp
 $Comp
-L GND #PWR04
+L GND #PWR12
 U 1 1 56BD6B31
 P 8100 5050
-F 0 "#PWR04" H 8100 4800 50  0001 C CNN
+F 0 "#PWR12" H 8100 4800 50  0001 C CNN
 F 1 "GND" H 8100 4900 50  0000 C CNN
 F 2 "" H 8100 5050 50  0000 C CNN
@@
 $EndComp
 $Comp
-L GND #PWR05
+L GND #PWR13
 U 1 1 56BD7318
 P 8500 5325
-F 0 "#PWR05" H 8500 5075 50  0001 C CNN
+F 0 "#PWR13" H 8500 5075 50  0001 C CNN
 F 1 "GND" H 8500 5175 50  0000 C CNN
 F 2 "" H 8500 5325 50  0000 C CNN
@@
 $EndComp
 $Comp
-L +5V #PWR06
+L +5V #PWR10
 U 1 1 56BDBA6B
 P 8000 3650
-F 0 "#PWR06" H 8000 3500 50  0001 C CNN
+F 0 "#PWR10" H 8000 3500 50  0001 C CNN
 F 1 "+5V" H 8000 3790 50  0000 C CNN
 F 2 "" H 8000 3650 50  0000 C CNN
@@
 147usec/inch
 $Comp
-L GND #PWR07
+L GND #PWR11
 U 1 1 56BDBACE
 P 8000 3925
-F 0 "#PWR07" H 8000 3925 30  0001 C CNN
+F 0 "#PWR11" H 8000 3925 30  0001 C CNN
 F 1 "GND" H 8000 3855 30  0001 C CNN
 F 2 "" H 8000 3925 60  0000 C CNN
@@
 $EndComp
 $Comp
-L GND #PWR08
+L GND #PWR2
 U 1 1 56B16EDA
 P 2450 2375
-F 0 "#PWR08" H 2450 2375 30  0001 C CNN
+F 0 "#PWR2" H 2450 2375 30  0001 C CNN
 F 1 "GND" H 2450 2305 30  0001 C CNN
 F 2 "" H 2450 2375 60  0000 C CNN
@@
 $EndComp
 $Comp
-L GND #PWR09
+L GND #PWR9
 U 1 1 56BD42F1
 P 7925 2275
-F 0 "#PWR09" H 7925 2025 50  0001 C CNN
+F 0 "#PWR9" H 7925 2025 50  0001 C CNN
 F 1 "GND" H 7925 2125 50  0000 C CNN
 F 2 "" H 7925 2275 50  0000 C CNN
@@
 $EndComp
 $Comp
-L SW_PUSH SW1
-U 1 1 56BEA4C8
-P 3425 1975
-F 0 "SW1" H 3575 2085 50  0000 C CNN
-F 1 "SW_PUSH" H 3425 1895 50  0000 C CNN
-F 2 "Buttons_Switches_ThroughHole:SW_TH_Tactile_Omron_B3F-10xx" H 3425 1975 50  0001 C CNN
-F 3 "" H 3425 1975 50  0000 C CNN
-	1    3425 1975
-	1    0    0    -1
-$EndComp
-$Comp
-L GND #PWR010
+L GND #PWR6
 U 1 1 56BEA5FD
-P 3850 2200
-F 0 "#PWR010" H 3850 2200 30  0001 C CNN
-F 1 "GND" H 3850 2130 30  0001 C CNN
-F 2 "" H 3850 2200 60  0000 C CNN
-F 3 "" H 3850 2200 60  0000 C CNN
-	1    3850 2200
+P 4025 2250
+F 0 "#PWR6" H 4025 2250 30  0001 C CNN
+F 1 "GND" H 4025 2180 30  0001 C CNN
+F 2 "" H 4025 2250 60  0000 C CNN
+F 3 "" H 4025 2250 60  0000 C CNN
+	1    4025 2250
 	-1   0    0    -1
 $EndComp
@@
 BW\n\nAN\nRX\nTX
 $Comp
-L +3.3V #PWR011
+L +3.3V #PWR1
 U 1 1 56B18BAE
 P 2450 1575
-F 0 "#PWR011" H 2450 1425 50  0001 C CNN
+F 0 "#PWR1" H 2450 1425 50  0001 C CNN
 F 1 "+3.3V" H 2450 1715 50  0000 C CNN
 F 2 "" H 2450 1575 50  0000 C CNN
@@
 NoConn ~ 1975 2475
 $Comp
-L PWR_FLAG #FLG012
+L PWR_FLAG #FLG1
 U 1 1 56BF040B
 P 2100 1650
-F 0 "#FLG012" H 2100 1745 50  0001 C CNN
+F 0 "#FLG1" H 2100 1745 50  0001 C CNN
 F 1 "PWR_FLAG" H 2100 1830 50  0000 C CNN
 F 2 "" H 2100 1650 50  0000 C CNN
@@
 $EndComp
 $Comp
-L PWR_FLAG #FLG013
+L PWR_FLAG #FLG2
 U 1 1 56BF0474
 P 3100 1625
-F 0 "#FLG013" H 3100 1720 50  0001 C CNN
+F 0 "#FLG2" H 3100 1720 50  0001 C CNN
 F 1 "PWR_FLAG" H 3100 1805 50  0000 C CNN
 F 2 "" H 3100 1625 50  0000 C CNN
@@
 $EndComp
 $Comp
-L PWR_FLAG #FLG014
+L PWR_FLAG #FLG3
 U 1 1 56BF0510
-P 4025 1975
-F 0 "#FLG014" H 4025 2070 50  0001 C CNN
-F 1 "PWR_FLAG" H 4025 2155 50  0000 C CNN
-F 2 "" H 4025 1975 50  0000 C CNN
-F 3 "" H 4025 1975 50  0000 C CNN
-	1    4025 1975
+P 4025 1875
+F 0 "#FLG3" H 4025 1970 50  0001 C CNN
+F 1 "PWR_FLAG" H 4025 2055 50  0000 C CNN
+F 2 "" H 4025 1875 50  0000 C CNN
+F 3 "" H 4025 1875 50  0000 C CNN
+	1    4025 1875
 	1    0    0    -1
 $EndComp
@@
 Text Notes 8150 3075 0    79   ~ 0
 Rangefinder
-Text Notes 2950 2475 0    79   ~ 0
+Text Notes 3050 2750 0    79   ~ 0
 Power Input\nand Return
 $Comp
@@
 $EndComp
 $Comp
-L GND #PWR015
+L GND #PWR4
 U 1 1 56BF43F4
 P 2825 4525
-F 0 "#PWR015" H 2825 4275 50  0001 C CNN
+F 0 "#PWR4" H 2825 4275 50  0001 C CNN
 F 1 "GND" H 2825 4375 50  0000 C CNN
 F 2 "" H 2825 4525 50  0000 C CNN
@@
 $EndComp
 $Comp
-L GND #PWR016
+L GND #PWR5
 U 1 1 56BF4462
 P 3175 4525
-F 0 "#PWR016" H 3175 4275 50  0001 C CNN
+F 0 "#PWR5" H 3175 4275 50  0001 C CNN
 F 1 "GND" H 3175 4375 50  0000 C CNN
 F 2 "" H 3175 4525 50  0000 C CNN
@@
 	2800 2175 1975 2175
 Wire Wire Line
-	1975 1975 3125 1975
+	1975 1975 3150 1975
 Wire Wire Line
 	4850 4375 5675 4375
@@
 	5950 5175 5950 4175
 Wire Wire Line
-	3725 1975 4025 1975
-Wire Wire Line
-	3850 1975 3850 2200
+	4025 1875 4025 2250
 Wire Wire Line
 	7925 2200 7925 2275
@@
 	2450 2275 2450 2375
 Connection ~ 2100 2275
-Connection ~ 3850 1975
 Wire Wire Line
 	2800 1700 3100 1700
@@
 	5800 2250 5800 2350
 $Comp
-L GND #PWR017
+L GND #PWR7
 U 1 1 56C1E93B
 P 5800 2350
-F 0 "#PWR017" H 5800 2100 50  0001 C CNN
+F 0 "#PWR7" H 5800 2100 50  0001 C CNN
 F 1 "GND" H 5800 2200 50  0000 C CNN
 F 2 "" H 5800 2350 50  0000 C CNN
@@
 Wire Wire Line
 	4850 3975 6250 3975
+Wire Wire Line
+	4025 1975 3750 1975
+Connection ~ 4025 1975
+NoConn ~ 3750 2075
+NoConn ~ 3150 2075
+$Comp
+L SW_PUSH_B3F_1XXX SW?
+U 1 1 56C77688
+P 3450 1975
+F 0 "SW?" H 3600 2085 50  0000 C CNN
+F 1 "SW_PUSH_B3F_1XXX" H 3420 1775 50  0000 C CNN
+F 2 "" H 3450 1975 50  0000 C CNN
+F 3 "" H 3450 1975 50  0000 C CNN
+	1    3450 1975
+	1    0    0    -1
+$EndComp
 $EndSCHEMATC
